Commit message: Fix robot

File: ex01/robot_description/urdf/robot.urdf.xacro (robot description, xacro)
@@ -1,7 +1,8 @@
 <?xml version="1.0" ?>
 <robot name='robot' xmlns:xacro="http://ros.org/wiki/xacro">
-    <xacro:include filename="$(find robot_description)/urdf/gazebo.urdf.xacro" />
-    <!--xacro:include filename="$(find robot_description)/urdf/lidar.urdf.xacro" /-->
-    <!--xacro:include filename="$(find robot_description)/urdf/depth.urdf.xacro" /-->
+    <xacro:include filename="gazebo.urdf.xacro" />
+    <xacro:include filename="lidar.urdf.xacro"/>
+    <xacro:include filename="depth.urdf.xacro" />
+    <xacro:include filename="imu.urdf.xacro" />
     <xacro:property name="chassis_length" value="0.335"/>
     <xacro:property name="chassis_width" value="0.265"/>

File: ex02/robot_description/urdf/robot.urdf.xacro (robot description, xacro)
@@ -1,7 +1,8 @@
 <?xml version="1.0" ?>
 <robot name='robot' xmlns:xacro="http://ros.org/wiki/xacro">
-    <xacro:include filename="$(find robot_description)/urdf/gazebo.urdf.xacro" />
-    <!--xacro:include filename="$(find robot_description)/urdf/lidar.urdf.xacro" /-->
-    <!--xacro:include filename="$(find robot_description)/urdf/depth.urdf.xacro" /-->
+    <xacro:include filename="gazebo.urdf.xacro" />
+    <xacro:include filename="lidar.urdf.xacro"/>
+    <xacro:include filename="depth.urdf.xacro" />
+    <xacro:include filename="imu.urdf.xacro" />
     <xacro:property name="chassis_length" value="0.335"/>
     <xacro:property name="chassis_width" value="0.265"/>

File: ex05/robot_description/urdf/robot.urdf.xacro (robot description, xacro)
@@ -1,7 +1,8 @@
 <?xml version="1.0" ?>
 <robot name='robot' xmlns:xacro="http://ros.org/wiki/xacro">
-    <xacro:include filename="$(find robot_description)/urdf/gazebo.urdf.xacro" />
-    <!--xacro:include filename="$(find robot_description)/urdf/lidar.urdf.xacro" /-->
-    <!--xacro:include filename="$(find robot_description)/urdf/depth.urdf.xacro" /-->
+    <xacro:include filename="gazebo.urdf.xacro" />
+    <xacro:include filename="lidar.urdf.xacro"/>
+    <xacro:include filename="depth.urdf.xacro" />
+    <xacro:include filename="imu.urdf.xacro" />
     <xacro:property name="chassis_length" value="0.335"/>
     <xacro:property name="chassis_width" value="0.265"/>
@@ -84,5 +85,5 @@
         <visual>
             <geometry>
-                <box size="${wheel_radius*2} ${wheel_radius*2} ${wheel_thickness}"/>
+                <cylinder radius="${wheel_radius}" length="${wheel_thickness}"/>
             </geometry>
             <material name="blue"/>
@@ -113,5 +114,5 @@
         <visual>
             <geometry>
-                <box size="${wheel_radius*2} ${wheel_radius*2} ${wheel_thickness}"/>
+                <cylinder radius="${wheel_radius}" length="${wheel_thickness}"/>
             </geometry>
             <material name="blue"/>

Commit message: Fix tasks

File: ex01/robot_description/urdf/robot.urdf.xacro (robot description, xacro)
@@ -1,8 +1,7 @@
 <?xml version="1.0" ?>
 <robot name='robot' xmlns:xacro="http://ros.org/wiki/xacro">
-    <xacro:include filename="gazebo.urdf.xacro" />
-    <xacro:include filename="lidar.urdf.xacro"/>
-    <xacro:include filename="depth.urdf.xacro" />
-    <xacro:include filename="imu.urdf.xacro" />
+    <xacro:include filename="$(find robot_description)/urdf/gazebo.urdf.xacro" />
+    <!--xacro:include filename="$(find robot_description)/urdf/lidar.urdf.xacro" /-->
+    <!--xacro:include filename="$(find robot_description)/urdf/depth.urdf.xacro" /-->
     <xacro:property name="chassis_length" value="0.335"/>
     <xacro:property name="chassis_width" value="0.265"/>

File: ex02/robot_description/urdf/robot.urdf.xacro (robot description, xacro)
@@ -1,8 +1,7 @@
 <?xml version="1.0" ?>
 <robot name='robot' xmlns:xacro="http://ros.org/wiki/xacro">
-    <xacro:include filename="gazebo.urdf.xacro" />
-    <xacro:include filename="lidar.urdf.xacro"/>
-    <xacro:include filename="depth.urdf.xacro" />
-    <xacro:include filename="imu.urdf.xacro" />
+    <xacro:include filename="$(find robot_description)/urdf/gazebo.urdf.xacro" />
+    <!--xacro:include filename="$(find robot_description)/urdf/lidar.urdf.xacro" /-->
+    <!--xacro:include filename="$(find robot_description)/urdf/depth.urdf.xacro" /-->
     <xacro:property name="chassis_length" value="0.335"/>
     <xacro:property name="chassis_width" value="0.265"/>

File: ex05/robot_description/urdf/robot.urdf.xacro (robot description, xacro)
@@ -1,8 +1,7 @@
 <?xml version="1.0" ?>
 <robot name='robot' xmlns:xacro="http://ros.org/wiki/xacro">
-    <xacro:include filename="gazebo.urdf.xacro" />
-    <xacro:include filename="lidar.urdf.xacro"/>
-    <xacro:include filename="depth.urdf.xacro" />
-    <xacro:include filename="imu.urdf.xacro" />
+    <xacro:include filename="$(find robot_description)/urdf/gazebo.urdf.xacro" />
+    <!--xacro:include filename="$(find robot_description)/urdf/lidar.urdf.xacro" /-->
+    <!--xacro:include filename="$(find robot_description)/urdf/depth.urdf.xacro" /-->
     <xacro:property name="chassis_length" value="0.335"/>
     <xacro:property name="chassis_width" value="0.265"/>
@@ -85,5 +84,5 @@
         <visual>
             <geometry>
-                <cylinder radius="${wheel_radius}" length="${wheel_thickness}"/>
+                <box size="${wheel_radius*2} ${wheel_radius*2} ${wheel_thickness}"/>
             </geometry>
             <material name="blue"/>
@@ -114,5 +113,5 @@
         <visual>
             <geometry>
-                <cylinder radius="${wheel_radius}" length="${wheel_thickness}"/>
+                <box size="${wheel_radius*2} ${wheel_radius*2} ${wheel_thickness}"/>
             </geometry>
             <material name="blue"/>
